Commit message: test(so101): drop shipped-config audit; ship kinematics-only URDF
Drop the unit test that read real configs/so101/so101.yaml (a shipped-artifact
audit, not a unit test — clean-checkout FileNotFoundError, diverges from piper).
Replace so101_new_calib.urdf with a kinematics-only derivative (no mesh deps),
sync pyproject package-data.

File: jiuwensymbiosis/adapters/so101/description/so101_new_calib.urdf (robot description, URDF)
Before this commit: robot so101_new_calib, 8 links, 7 joints
Links:
- removed link moving_jaw_so101_v1_link
- link base_link: mass 0.147 -> None; geometry 
- link gripper_frame_link: mass 1e-9 -> None
- link gripper_link: mass 0.087 -> None; geometry 
- link lower_arm_link: mass 0.104 -> None; geometry 
- link shoulder_link: mass 0.100006 -> None; geometry 
- link upper_arm_link: mass 0.103 -> None; geometry 
- link wrist_link: mass 0.079 -> None; geometry 
Joints:
- removed joint gripper
- joint gripper_frame_joint: axis 0 0 0 -> (none)
